Commit message: Added launch files, fixed formatting errors for rviz (joint limits) in turtle_bot.urdf.xacro

File: turtle_brick/urdf/turtle_bot.urdf (robot description, URDF)
Before this commit: robot turtle-bot, 5 links, 4 joints
Links:
- link base_link: geometry collision box size=2.0 2.0 2.0; visual box size=2.0 2.0 2.0
- link fixed_link: geometry collision cylinder length=2.0 radius=0.2; visual cylinder length=2.0 radius=0.2
- link stem_link: geometry collision cylinder length=-1.0 radius=0.65; visual cylinder length=1.0 radius=0.5
Joints:
- joint fixed_joint: origin xyz=0 0 2.25 rpy=0 0 0 -> xyz=0 0 2.0 rpy=0 0 0
- joint platform_joint: limit effort=100 velocity=100 -> lower=0 upper=6.283185307179586 effort=100 velocity=100; origin xyz=0 0 1.25 rpy=0 0 0 -> xyz=0 0 1.0 rpy=0 0 0
- joint stem_joint: limit effort=100 velocity=100 -> lower=0 upper=6.283185307179586 effort=100 velocity=100; origin xyz=0 0 -1 rpy=0 0 0 -> xyz=0 0 -1.0 rpy=0 0 0
- joint wheel_joint: limit effort=100 velocity=100 -> lower=0 upper=6.283185307179586 effort=100 velocity=100; origin xyz=0 0 -2.2 rpy=0 0 0 -> xyz=0 0 -3.0 rpy=0 0 0

File: turtle_brick/urdf/turtle_bot.urdf.xacro (robot description, xacro)
@@ -1,8 +1,13 @@
 <robot name="turtle-bot" xmlns:xacro="http://www.ros.org/wiki/xacro">
     <xacro:include filename="materials.urdf.xacro"/>
+    <xacro:property name="turtle_config" value="${xacro.load_yaml('$(find turtle_brick)/config/turtle.yaml')}"/>
+    <xacro:property name="wheel_radius" value="${turtle_config['dimensions']['wheel_radius']}"/>
+    <xacro:property name="platform_height" value="${turtle_config['dimensions']['platform_height'] - wheel_radius*2}"/>
+    <xacro:property name="fixed_length" value="${0.4*platform_height}" />
+    <xacro:property name="base_length" value="${0.4*platform_height}" />
     <link name="base_link">
         <visual>
             <geometry>
-                <box size="2 2 2" />
+                <box size="${base_length} ${base_length} ${base_length}" />
             </geometry>
             <material name="green"/>
@@ -10,9 +15,8 @@
         <collision>
             <geometry>
-                <box size="2 2 2" />
+                <box size="${base_length} ${base_length} ${base_length}" />
             </geometry>
         </collision>
     </link>
-    <xacro:property name="fixed_length" value="2.5" />
     <link name="fixed_link">
         <visual>
@@ -30,9 +34,10 @@
         </collision>
     </link>
+    <xacro:property name="platform_length" value="0.2" />
     <link name="platform_link">
         <visual>
-            <origin xyz="0 0 0" rpy="0 0 0"/>
+            <origin xyz="0 0 ${platform_length/2}" rpy="0 0 0"/>
             <geometry>
-                <cylinder length="0.2" radius="2"/>
+                <cylinder length="${platform_length}" radius="2"/>
             </geometry>
             <material name="blue"/>
@@ -41,14 +46,14 @@
             <origin xyz="0 0 0" rpy="0 0 0" />
             <geometry>
-                <cylinder length="0.2" radius="2"/>
+                <cylinder length="${platform_length}" radius="2"/>
             </geometry>
         </collision>
     </link>
-    <xacro:property name="stem_length" value="0.4"/>
+    <xacro:property name="stem_length" value="${platform_height*0.2}"/>
     <link name="stem_link">
         <visual>
-            <origin xyz="0 0 0" rpy="0 0 0" />
+            <origin xyz="0 0 ${-stem_length/2}" rpy="0 0 0" />
             <geometry>
-                <cylinder length="${-stem_length}" radius="0.5"/>
+                <cylinder length="${stem_length}" radius="0.5"/>
             </geometry>
             <material name="orange"/>
@@ -57,9 +62,8 @@
             <origin xyz="0 0 0" rpy="0 0 0" />
             <geometry>
-                <cylinder length="-0.4" radius="0.65"/>
+                <cylinder length="${-stem_length}" radius="0.65"/>
             </geometry>
         </collision>
     </link>
-    <xacro:property name="wheel_radius" value="2"/>
     <xacro:property name="wheel_length" value="0.5"/>
     <link name="wheel_link">
@@ -79,5 +83,5 @@
     </link>
     <joint name="fixed_joint" type="fixed">
-        <origin xyz="0 0 ${fixed_length/2 + 1}" rpy="0 0 0"/>
+        <origin xyz="0 0 ${fixed_length/2 + base_length/2}" rpy="0 0 0"/>
         <parent link="base_link"/>
         <child link="fixed_link"/>
@@ -88,19 +92,19 @@
         <child link="platform_link"/>
         <axis xyz="1 0 0"/>
-        <limit effort="100" velocity="100"/>
+        <limit lower="0" upper="${pi*2}" effort="100" velocity="100"/>
     </joint>
     <joint name="stem_joint" type="revolute">
-        <origin xyz="0 0 -1" rpy="0 0 0"/>
+        <origin xyz="0 0 ${-base_length/2}" rpy="0 0 0"/>
         <parent link="base_link"/>
         <child link="stem_link"/>
         <axis xyz="0 0 1"/>
-        <limit effort="100" velocity="100"/>
+        <limit lower="0" upper="${pi*2}" effort="100" velocity="100"/>
     </joint>
     <joint name="wheel_joint" type="revolute">
-        <origin xyz="0 0 ${-wheel_radius-0.2}" rpy="0 0 0" />
+        <origin xyz="0 0 ${-wheel_radius-stem_length}" rpy="0 0 0" />
         <parent link="stem_link"/>
         <child link="wheel_link"/>
         <axis xyz="1 0 0"/>
-        <limit effort="100" velocity="100"/>
+        <limit lower="0" upper="${pi*2}" effort="100" velocity="100"/>
     </joint>
 </robot>
