Commit message: Created-operational-tf-tree-and-updated-rviz-file

File: turtle_brick/urdf/turtle_bot.urdf.xacro (robot description, xacro)
@@ -4,5 +4,5 @@
     <xacro:property name="wheel_radius" value="${turtle_config['dimensions']['wheel_radius']}"/>
     <xacro:property name="platform_height" value="${turtle_config['dimensions']['platform_height'] - wheel_radius*2}"/>
-    <xacro:property name="fixed_length" value="${0.4*platform_height}" />
+    <xacro:property name="cylinder_length" value="${0.4*platform_height}" />
     <xacro:property name="base_length" value="${0.4*platform_height}" />
     <link name="base_link">
@@ -19,9 +19,9 @@
         </collision>
     </link>
-    <link name="fixed_link">
+    <link name="cylinder_link">
         <visual>
             <origin xyz="0 0 0" rpy="0 0 0"/>
             <geometry>
-                <cylinder length="${fixed_length}" radius="0.2"/>
+                <cylinder length="${cylinder_length}" radius="0.2"/>
             </geometry>
             <material name="white"/>
@@ -30,5 +30,5 @@
             <origin xyz="0 0 0" rpy="0 0 0" />
             <geometry>
-                <cylinder length="${fixed_length}" radius="0.2" />
+                <cylinder length="${cylinder_length}" radius="0.2" />
             </geometry>
         </collision>
@@ -82,12 +82,12 @@
         </collision>
     </link>
-    <joint name="fixed_joint" type="fixed">
-        <origin xyz="0 0 ${fixed_length/2 + base_length/2}" rpy="0 0 0"/>
+    <joint name="cylinder_joint" type="fixed">
+        <origin xyz="0 0 ${cylinder_length/2 + base_length/2}" rpy="0 0 0"/>
         <parent link="base_link"/>
-        <child link="fixed_link"/>
+        <child link="cylinder_link"/>
     </joint>
     <joint name="platform_joint" type="revolute">
-        <origin xyz="0 0 ${fixed_length/2}" rpy="0 0 0"/>
-        <parent link="fixed_link"/>
+        <origin xyz="0 0 ${cylinder_length/2}" rpy="0 0 0"/>
+        <parent link="cylinder_link"/>
         <child link="platform_link"/>
         <axis xyz="1 0 0"/>

Commit message: Added joint_status and made the stem_link move in the direction of movement. Made the wheel rotate. Started formatting arena.py and Place.srv.

File: turtle_brick/urdf/turtle_bot.urdf.xacro (robot description, xacro)
@@ -2,6 +2,6 @@
     <xacro:include filename="materials.urdf.xacro"/>
     <xacro:property name="turtle_config" value="${xacro.load_yaml('$(find turtle_brick)/config/turtle.yaml')}"/>
-    <xacro:property name="wheel_radius" value="${turtle_config['dimensions']['wheel_radius']}"/>
-    <xacro:property name="platform_height" value="${turtle_config['dimensions']['platform_height'] - wheel_radius*2}"/>
+    <xacro:property name="wheel_radius" value="${turtle_config['turtle_robot']['ros__parameters']['wheel_radius']}"/>
+    <xacro:property name="platform_height" value="${turtle_config['turtle_robot']['ros__parameters']['platform_height'] - wheel_radius*2}"/>
     <xacro:property name="cylinder_length" value="${0.4*platform_height}" />
     <xacro:property name="base_length" value="${0.4*platform_height}" />

Commit message: Updated arena.py and xacro to move odom and world to ground while tracking base_link Added brick catching and brick carrying capabilities

File: turtle_brick/urdf/turtle_bot.urdf.xacro (robot description, xacro)
@@ -4,6 +4,6 @@
     <xacro:property name="wheel_radius" value="${turtle_config['turtle_robot']['ros__parameters']['wheel_radius']}"/>
     <xacro:property name="platform_height" value="${turtle_config['turtle_robot']['ros__parameters']['platform_height'] - wheel_radius*2}"/>
-    <xacro:property name="cylinder_length" value="${0.4*platform_height}" />
-    <xacro:property name="base_length" value="${0.4*platform_height}" />
+    <xacro:property name="base_length" value="1" />
+    <xacro:property name="cylinder_length" value="${platform_height-1.4}" />
     <link name="base_link">
         <visual>
@@ -50,5 +50,5 @@
         </collision>
     </link>
-    <xacro:property name="stem_length" value="${platform_height*0.2}"/>
+    <xacro:property name="stem_length" value="0.2"/>
     <link name="stem_link">
         <visual>

Commit message: Debugged problems: - Made brick also rotate in the Slide - Fixed Wheel Slide Issue - Fixed config/turtle.yaml - Fixed physics file bugs

File: turtle_brick/urdf/turtle_bot.urdf.xacro (robot description, xacro)
@@ -2,6 +2,6 @@
     <xacro:include filename="materials.urdf.xacro"/>
     <xacro:property name="turtle_config" value="${xacro.load_yaml('$(find turtle_brick)/config/turtle.yaml')}"/>
-    <xacro:property name="wheel_radius" value="${turtle_config['turtle_robot']['ros__parameters']['wheel_radius']}"/>
-    <xacro:property name="platform_height" value="${turtle_config['turtle_robot']['ros__parameters']['platform_height'] - wheel_radius*2}"/>
+    <xacro:property name="wheel_radius" value="${turtle_config['/**']['ros__parameters']['wheel_radius']}"/>
+    <xacro:property name="platform_height" value="${turtle_config['/**']['ros__parameters']['platform_height'] - wheel_radius*2}"/>
     <xacro:property name="base_length" value="1" />
     <xacro:property name="cylinder_length" value="${platform_height-1.4}" />

Commit message: Fixed issue with gui and jsp in xml launch files

File: turtle_brick/urdf/turtle_bot.urdf.xacro (robot description, xacro)
@@ -62,5 +62,5 @@
             <origin xyz="0 0 0" rpy="0 0 0" />
             <geometry>
-                <cylinder length="${-stem_length}" radius="0.65"/>
+                <cylinder length="${-stem_length}" radius="0.5"/>
             </geometry>
         </collision>
